File: shift-register-breakout-pcb.kicad_pcb (KiCad board)
At the start: 2 copper layers, 75 x 25 mm, 27 parts, among them J1 Conn_01x08_Socket, J2 Conn_01x08_Socket, J3 Conn_01x08_Socket, J4 Conn_01x08_Socket, J5 Conn_01x08_Socket, J6 Conn_01x03_Socket, J7 vik-module-connector

Commit message: final vik version
Parts:
- removed LOGO3: **REF, ct-kicad:qmk-lite
- added FID2: Fiducial, vik:vik-logo-small, B.Cu at (139.3, 85.3)
- added J8: Conn_01x04_Socket, Connector_JST:JST_XH_B4B-XH-A_1x04_P2.50mm_Vertical, F.Cu at (134.7, 71.3)
- added LOGO2: **REF, ct-kicad:shift-reg-qr-10mm, B.Cu at (84.6, 72.0)
- J1: value Conn_01x08_Socket -> Conn_01x04_Socket; footprint Connector_PinSocket_2.54mm:PinSocket_1x08_P2.54mm_Vertical -> Connector_JST:JST_XH_B4B-XH-A_1x04_P2.50mm_Vertical
- J2, J3, J4, J5: footprint Connector_JST:JST_EH_B8B-EH-A_1x08_P2.50mm_Vertical -> Connector_JST:JST_XH_B8B-XH-A_1x08_P2.50mm_Vertical
- moved LOGO1 66.1 mm to (74.9, 71.2)
- moved H1 60.1 mm to (75.0, 65.0)
- moved R4 51.7 mm to (125.4, 87.3), turned to -90 degrees
- moved REG-COL4 45.8 mm to (121.9, 71.3), turned to 0 degrees
- moved H2 40.1 mm to (140.0, 65.0)
- moved R2 38.8 mm to (125.4, 80.5), turned to -90 degrees
- moved J3 32.8 mm to (75.6, 85.7)
- moved J2 32.6 mm to (75.6, 78.9)
- moved C5 28.9 mm to (106.8, 65.8), turned to 90 degrees
- moved REG-ROW2 27.7 mm to (94.8, 71.1)
- moved C6 27.7 mm to (117.5, 65.9), turned to 90 degrees
- moved C3 26.3 mm to (90.4, 65.8)
- moved REG-ROW1 26.2 mm to (84.3, 71.2)
- moved C1 24.6 mm to (79.8, 65.8)
- moved REG-COL3 23.8 mm to (111.2, 71.3), turned to 0 degrees
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Connections:
- J1 pad 1: GND -> SPI_CLK
- J1 pad 2: +3V3 -> COL_CS
- J1 pad 3: SPI_MOSI -> SPI_MISO
- J1 pad 4: ROW_CS -> COL_LATCH
Routing:
- net +3V3: track 145.0 -> 99.4 mm, vias 12 -> 7
- net Net-(J6-Pin_2): track 64.6 -> 23.0 mm
- net SPI_MOSI: track 32.8 -> 71.1 mm, vias 2 -> 4
- net COL_LATCH: track 9.58 -> 43.5 mm, vias 1 -> 3
- net COL_CS_MOS: track 65.5 -> 35.5 mm, vias 5 -> 3
- net ROW_CS: track 55.9 -> 83.9 mm, vias 6 -> 5
- net COL_CS: track 82.7 -> 56.3 mm, vias 8 -> 6
- net Net-(REG-COL3-SA): track 0.00 -> 23.6 mm, vias 0 -> 2
- net col6: track 35.1 -> 15.1 mm, vias 1 -> 2
- net col11: track 11.1 -> 30.1 mm
- net col12: track 9.83 -> 28.8 mm
- net col10: track 12.3 -> 28.5 mm
- net SPI_CLK: track 109.4 -> 93.3 mm, vias 14 -> 5
- net row10: track 45.1 -> 29.2 mm, vias 6 -> 2
- net col13: track 8.81 -> 24.6 mm
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Other:
- board size 75 x 25 mm -> 75 x 30 mm
- board text added: ".C"
- board text added: "CL"
- board text added: "CS"
- board text added: "CS.R"
- board text added: "ENABLE LATCH"
- board text added: "L"
- board text added: "LA"
- board text added: "MI"
- board text added: "MO"
- board text added: "Rw.8"
- board text added: "VIK interconnect"
- board text added: "v2.0"
- board text removed: "C.CS"
- board text removed: "CLK"
- board text removed: "COL_CS JOIN"
- board text removed: "DIODE: ROW2COL"
- board text removed: "Hole: M2"
- board text removed: "LATCH"
- board text removed: "LATCH ENABLE"
- board text removed: "MISO"
- board text removed: "MOSI"
- board text removed: "R.CS"
- board text removed: "Rw.15"
- board text removed: "v1.0"
- board text removed: "v1.1"
